Commit message: changed URDF for the cartesian control

File: demo/SO100/URDF/so100_original.urdf (robot description, URDF)
Before this commit: robot so_arm100, 7 links, 6 joints
Joints:
- joint elbow_flex: axis 0 1 0 -> 1 0 0; limit lower=-3.14158 upper=3.14159 effort=35 velocity=1 -> lower=-3.14158 upper=0 effort=35 velocity=1; origin xyz=0 0 0.113 rpy=0 0 0 -> xyz=0 0.11257 0.028 rpy=1.57079 0 0
- joint gripper: origin xyz=0 0 0 rpy=0 0 0 -> xyz=-0.0202 -0.0244 0 rpy=0 3.14158 0
- joint shoulder_lift: axis 0 1 0 -> 1 0 0; limit lower=-3.14159 upper=3.14159 effort=35 velocity=1 -> lower=0 upper=3.5 effort=35 velocity=1; origin xyz=0 0 0.105 rpy=0 0 0 -> xyz=0 0.1025 0.0306 rpy=-1.8 0 0
- joint shoulder_pan: axis 0 0 1 -> 0 1 0; limit lower=-3.14159 upper=3.14159 effort=35 velocity=1 -> lower=-2 upper=2 effort=35 velocity=1; origin xyz=0 -0.0452 0.0165 rpy=0 0 0 -> xyz=0 -0.0452 0.0165 rpy=1.57079 0 0
- joint wrist_flex: axis 0 1 0 -> 1 0 0; limit lower=-3.14159 upper=3.14159 effort=35 velocity=1 -> lower=-2.5 upper=1.2 effort=35 velocity=1; origin xyz=0 0 0.1349 rpy=0 0 0 -> xyz=0 0.0052 0.1349 rpy=-1 0 0
- joint wrist_roll: axis 0 0 1 -> 0 1 0; origin xyz=0 0 0.0601 rpy=0 0 0 -> xyz=0 -0.0601 0 rpy=0 1.57079 0
